File: hw/power.sch (KiCad schematic (older format))
At the start: 18 parts, among them J4 POWER, U8 MCP16301H, U9 MCP1826S

Commit message: updated schematic
Parts:
- removed D6: D_Bridge_+-AA, symbol D_Bridge_+-AA
- added D6, D7: SK32SMA, symbol D_Schottky
- D8: renamed from D7; value SS14 -> SK32SMA
- D9: renamed from D8; value SS14 -> SK32SMA
- renumbered C15 to C17, C16 to C18, C17 to C19, C18 to C20, C19 to C21, C20 to C22, C21 to C23, C22 to C24, C23 to C25, R9 to R18, R10 to R19, U9 to U10, U8 to U9
Connections:
- net GND: now also J4.1 (Pin_1)
- net VCC: now also D6.1 (K), D7.2 (A); no longer C17.1, C18.1, C19.1, U9.4 (EN), U9.5 (VIN)
- net at J4.2 (Pin_2): now also D6.2 (A)
- new net: C17.1, C18.1, C19.1, D7.1 (K), U9.4 (EN), U9.5 (VIN)
Other:
- moved on the sheet: J4
