File: hw/arcar.kicad_pcb (KiCad board)
At the start: 2 copper layers, 60 x 36 mm, 55 parts, among them J1 USB_B_Micro, J2 MOTOR, J3 POWER, M1 screw, M2 screw, P1 AVR_ISP_02X03, SW1 SW_Push, U1 USBLC6-2SC6, U2 ATMEGA328PB-AU, U3 CP2102, U4 ULN2003A, U5 LSM9DS1, U6 TLE52062GAUMA1, U7 RN4871, U8 MCP1804T-3302I/DB

Commit message: change LED resistors
Parts:
- R10, R6, R7, R8: value 330R -> 1k
Changed lines of the file:
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@@
       (effects (font (size 1 1) (thickness 0.15)) (justify mirror))
     )
-    (fp_text value 330R (at 0 -1.75 270) (layer B.Fab)
+    (fp_text value 1k (at 0 -1.75 270) (layer B.Fab)
       (effects (font (size 1 1) (thickness 0.15)) (justify mirror))
     )
@@
       (effects (font (size 1 1) (thickness 0.15)) (justify mirror))
     )
-    (fp_text value 330R (at 0 -1.75 270) (layer B.Fab)
+    (fp_text value 1k (at 0 -1.75 270) (layer B.Fab)
       (effects (font (size 1 1) (thickness 0.15)) (justify mirror))
     )
@@
       (effects (font (size 1 1) (thickness 0.15)) (justify mirror))
     )
-    (fp_text value 330R (at 0 -1.75 270) (layer B.Fab)
+    (fp_text value 1k (at 0 -1.75 270) (layer B.Fab)
       (effects (font (size 1 1) (thickness 0.15)) (justify mirror))
     )
@@
       (effects (font (size 1 1) (thickness 0.15)) (justify mirror))
     )
-    (fp_text value 330R (at 0 -1.75 270) (layer B.Fab)
+    (fp_text value 1k (at 0 -1.75 270) (layer B.Fab)
       (effects (font (size 1 1) (thickness 0.15)) (justify mirror))
     )
